File: board_sch/rx5usb_board.kicad_pcb (KiCad board)
At the start: 2 copper layers, 112 x 80 mm, 14 parts, among them P1 RX5_WDC, SW1 SWITCH_INV, U1 TEENSYPP2, U2 39SF040

Commit message: Rename footprints
Parts:
- C1: footprint rx5usb:C2V8 -> rx5usb:C1
- D1: footprint rx5usb:D4 -> rx5usb:1N5817
- D3, D4: footprint rx5usb:D3 -> rx5usb:1N4148
- R1, R2, R3, R4: footprint rx5usb:R4-LARGE_PADS -> rx5usb:RESISTOR
